File: fuente-12v.kicad_pcb (KiCad board)
At the start: 2 copper layers, 150 x 80 mm, 89 parts, among them J1 Conn_01x03_Pin, J2 Screw_Terminal_01x03, J3 Conn_01x02_Pin, J5 OUTPUT, J6 Screw_Terminal_01x03 P5mm, Q1 IPP65R190C7, Q2 CSD16403Q5A, U1 UCC287501D, U2 TCMT1107, U3 TL432DBZ, U4 TPS24701DGKR, U5 NE555P

Commit message: Fixes
Parts:
- R15, R16: value 1 -> 0.018
- moved D6 5.08 mm to (184.2, 114.0), turned to 180 degrees
Other:
- outline, holes or cut-outs redrawn
- board text added: "110V - 240V"
- board text added: "Fuente Flyback 12V 2.5A Proyecto Electrónica de Potenica 2025"
Changed lines of the file:
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@@
 	(footprint "Package_TO_SOT_THT:TO-220-3_Vertical"
 		(layer "F.Cu")
-		(at 179.17 114)
+		(at 184.25 114 180)
 		(descr "TO-220-3, Vertical, RM 2.54mm, see https://www.vishay.com/docs/66542/to-220-1.pdf, generated with kicad-footprint-generator TO_SOT_THT_generate.py")
 		(tags "TO-220-3 Vertical RM 2.54mm")
@@
 		(attr through_hole)
 		(fp_line
-			(start -2.57 -3.26)
-			(end 7.65 -3.26)
+			(start 7.65 1.36)
+			(end -2.57 1.36)
 			(stroke
 				(width 0.12)
@@
 		)
 		(fp_line
-			(start -2.57 -1.88)
-			(end 7.65 -1.88)
+			(start 7.65 -3.26)
+			(end 7.65 1.36)
 			(stroke
 				(width 0.12)
@@
 		)
 		(fp_line
-			(start -2.57 1.36)
-			(end -2.57 -3.26)
+			(start 4.39 -3.26)
+			(end 4.39 -1.88)
 			(stroke
 				(width 0.12)
@@
 		)
 		(fp_line
-			(start 4.39 -3.26)
-			(end 4.39 -1.88)
+			(start -2.57 1.36)
+			(end -2.57 -3.26)
 			(stroke
 				(width 0.12)
@@
 		)
 		(fp_line
-			(start 7.65 -3.26)
-			(end 7.65 1.36)
+			(start -2.57 -1.88)
+			(end 7.65 -1.88)
 			(stroke
 				(width 0.12)
@@
 		)
 		(fp_line
-			(start 7.65 1.36)
-			(end -2.57 1.36)
+			(start -2.57 -3.26)
+			(end 7.65 -3.26)
 			(stroke
 				(width 0.12)
@@
 		)
 		(fp_line
-			(start -2.46 -1.88)
-			(end 7.54 -1.88)
+			(start 4.39 -3.15)
+			(end 4.39 -1.88)
 			(stroke
 				(width 0.1)
@@
 		)
 		(fp_line
-			(start 4.39 -3.15)
-			(end 4.39 -1.88)
+			(start -2.46 -1.88)
+			(end 7.54 -1.88)
 			(stroke
 				(width 0.1)
@@
 		)
 		(pad "1" thru_hole rect
-			(at 0 0)
+			(at 0 0 180)
 			(size 1.905 2)
 			(drill 1.1)
@@
 		)
 		(pad "2" thru_hole oval
-			(at 2.54 0)
+			(at 2.54 0 180)
 			(size 1.905 2)
 			(drill 1.1)
@@
 		)
 		(pad "3" thru_hole oval
-			(at 5.08 0)
+			(at 5.08 0 180)
 			(size 1.905 2)
 			(drill 1.1)
@@
 			)
 		)
-		(property "Value" "1"
+		(property "Value" "0.018"
 			(at 0 -2.63 90)
 			(layer "B.Fab")
@@
 			)
 		)
-		(property "Value" "1"
+		(property "Value" "0.018"
 			(at 0 -2.63 90)
 			(layer "B.Fab")
@@
 	)
 	(gr_arc
-		(start 167.5 58.5)
-		(mid 168.5 57.5)
-		(end 169.5 58.5)
+		(start 167.5 86.5)
+		(mid 168.5 85.5)
+		(end 169.5 86.5)
 		(stroke
 			(width 0.2)
@@
 		(layer "Edge.Cuts")
 	)
+	(gr_line
+		(start 169.5 86.5)
+		(end 169.5 128.25)
+		(stroke
+			(width 0.2)
+			(type default)
+		)
+		(layer "Edge.Cuts")
+	)
 	(gr_rect
 		(start 70 55)
@@
 	)
 	(gr_arc
+		(start 169.5 77.5)
+		(mid 168.5 78.5)
+		(end 167.5 77.5)
+		(stroke
+			(width 0.2)
+			(type solid)
+		)
+		(layer "Edge.Cuts")
+	)
+	(gr_arc
+		(start 167.5 60)
+		(mid 168.5 59)
+		(end 169.5 60)
+		(stroke
+			(width 0.2)
+			(type solid)
+		)
+		(layer "Edge.Cuts")
+	)
+	(gr_arc
 		(start 169.5 128.25)
 		(mid 168.5 129.25)
@@
 	)
 	(gr_line
-		(start 167.5 128.25)
-		(end 167.5 58.5)
+		(start 167.5 86.5)
+		(end 167.5 128.25)
 		(stroke
 			(width 0.2)
@@
 	)
 	(gr_line
-		(start 169.5 58.5)
-		(end 169.5 128.25)
+		(start 167.5 77.5)
+		(end 167.5 60)
+		(stroke
+			(width 0.2)
+			(type default)
+		)
+		(layer "Edge.Cuts")
+	)
+	(gr_line
+		(start 169.5 60)
+		(end 169.5 77.5)
 		(stroke
 			(width 0.2)
@@
 		)
 	)
+	(gr_text "110V - 240V"
+		(at 72 114 0)
+		(layer "F.SilkS")
+		(effects
+			(font
+				(size 2 2)
+				(thickness 0.5)
+				(bold yes)
+			)
+			(justify left bottom)
+		)
+	)
 	(gr_text "G"
 		(at 70.35278 104.98889 270)
@@
 		)
 	)
+	(gr_text "Fuente Flyback 12V 2.5A\nProyecto Electrónica de\nPotenica   2025"
+		(at 79 70 0)
+		(layer "F.SilkS")
+		(effects
+			(font
+				(size 2 2)
+				(thickness 0.5)
+				(bold yes)
+			)
+			(justify left bottom)
+		)
+	)
 	(via
 		(at 215 60)
@@
 		(layers "F.Cu" "B.Cu")
 		(free yes)
+		(tenting none)
 		(net 0)
 	)
@@
 		(layers "F.Cu" "B.Cu")
 		(free yes)
+		(tenting none)
 		(net 0)
 	)
@@
 		(layers "F.Cu" "B.Cu")
 		(free yes)
+		(tenting none)
 		(net 0)
 	)
@@
 		(layers "F.Cu" "B.Cu")
 		(free yes)
+		(tenting none)
 		(net 0)
 	)
@@
 		(polygon
 			(pts
-				(xy 165 127.5) (xy 165 127.5) (xy 166.5 126) (xy 166.5 113) (xy 165 111.5) (xy 165 111.5) (xy 164 110.5)
-				(xy 126.25 110.5) (xy 125.75 110) (xy 122.75 110) (xy 122 110.75) (xy 104.75 110.75) (xy 92.5 123)
-				(xy 92.5 131) (xy 93.25 131.75) (xy 160.75 131.75)
+				(xy 165 127.5) (xy 166.5 126) (xy 166.5 113) (xy 165 111.5) (xy 164 110.5) (xy 126.25 110.5) (xy 125.75 110)
+				(xy 122.75 110) (xy 122 110.75) (xy 104.75 110.75) (xy 92.5 123) (xy 92.5 131) (xy 93.25 131.75)
+				(xy 160.75 131.75)
 			)
 		)

Commit message: Terminada. Necesita revision
Parts:
- added H1: MountingHole, MountingHole:MountingHole_4.3mm_M4_DIN965, F.Cu at (75.0, 130.0)
- added H2: MountingHole, MountingHole:MountingHole_4.3mm_M4_DIN965, F.Cu at (75.0, 55.0)
- added H3: MountingHole, MountingHole:MountingHole_4.3mm_M4_DIN965, F.Cu at (215.0, 130.0)
- added H4: MountingHole, MountingHole:MountingHole_4.3mm_M4_DIN965, F.Cu at (215.0, 55.0)
- added TP10: TestPoint, Connector_PinHeader_1.00mm:PinHeader_1x01_P1.00mm_Vertical, F.Cu at (134.5, 103.5)
- added TP11: TestPoint, Connector_PinHeader_1.00mm:PinHeader_1x01_P1.00mm_Vertical, F.Cu at (154.2, 109.8)
- added TP4: TestPoint, Connector_PinHeader_1.00mm:PinHeader_1x01_P1.00mm_Vertical, F.Cu at (139.5, 107.0)
- R2: renamed from R24; moved to B.Cu
- moved TP7 29.8 mm to (209.8, 114.0)
- moved R4 28.7 mm to (143.4, 88.6), turned to 90 degrees
- moved C14 25.1 mm to (146.4, 88.6), turned to 90 degrees
- moved R10 23.7 mm to (145.0, 84.0), turned to 0 degrees
- moved TP5 17.2 mm to (191.8, 114.0)
- moved D4 15.4 mm to (147.1, 80.2), turned to 0 degrees
- moved TP6 14.7 mm to (133.5, 107.5)
- moved R2 11.9 mm to (194.8, 92.8), turned to -90 degrees
- moved C8 8.11 mm to (136.5, 99.1), turned to 90 degrees
- moved TP8 5.75 mm to (171.8, 113.8)
- moved TP9 5.75 mm to (165.2, 113.8)
- moved TP3 4.79 mm to (207.6, 87.9)
- renumbered C8 to C1, C22 to C10, C16 to C11, C3 to C13, C24 to C14, C2 to C15, C7 to C16, C1 to C17, C19 to C18, C9 to C19, C29 to C2, C10 to C20, C11 to C21, C21 to C22, C27 to C23, C15 to C24, C13 to C25, C23 to C26, C17 to C3, C5 to C4, C25 to C5, C20 to C6, C26 to C7, C14 to C8, C4 to C9, D9 to D1, D6 to D2, D1 to D3, D8 to D4, D4 to D5, D5 to D6, D2 to D8, D3 to D9, J2 to J1, J6 to J2, J1 to J3, J5 to J4, J3 to J5, R17 to R1, R22 to R10, R6 to R11, R3 to R12, R18 to R13, R19 to R14, R7 to R15, R9 to R16, R10 to R17, R12 to R18, R11 to R19, R8 to R20, R5 to R21, R21 to R22, R20 to R23, R2 to R24, R4 to R25, RA1 to R27, RB1 to R28, R1 to R3, R23 to R4, R16 to R5, R13 to R6, R14 to R7, R15 to R8, R27 to R9, RV2 to RV1, RV1 to RV2, TP3 to TP2, TP6 to TP3, TP2 to TP6, TP8 to TP7, TP9 to TP8, TP7 to TP9, U5 to U1, U4 to U2, U2 to U4, U1 to U5
Connections:
- U1 pad 4: /5V -> +5V
Routing:
- net P_GND: track 177.5 -> 126.1 mm, vias 36 -> 50
- net /LINE_DC: track 96.8 -> 59.8 mm
- net Net-(U3-REF): track 18.3 -> 44.6 mm
- net /12V: track 156.6 -> 142.6 mm
- net +5V: track 35.9 -> 49.8 mm
- net Net-(D3-A): track 2.22 -> 15.5 mm, vias 0 -> 1
- net Net-(J3-Pin_2): track 15.6 -> 26.3 mm
- net /AUX_DRV: track 53.7 -> 64.4 mm
- net Net-(D6-A): track 22.4 -> 33.1 mm
- net Net-(D6-K): track 50.8 -> 59.5 mm
- net /VOUT: track 6.65 -> 14.6 mm
- net Net-(Q1-S): track 16.6 -> 24.3 mm
- net /FB: track 9.80 -> 15.5 mm
- net Net-(R17-Pad2): track 8.35 -> 14.1 mm
- net Net-(D2-A-Pad1): track 54.4 -> 59.2 mm
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Other:
- board size 150 x 80 mm -> 150 x 85 mm
- board text added: "CS"
- board text added: "DC"
- board text added: "DC_IN"
- board text added: "EXT"
- board text added: "FB"
- board text added: "GATE"
- board text added: "NORMAL"
- board text added: "OPTO LED"
- board text added: "Pedro Lauckner Bruno Glecer Nicolas Taurozzi Joaquín Cibeira"
- board text added: "SEC"
- board text added: "VAUX"
- board text added: "VDD"
- board text added: "VOUT"
- board text added: "VREF"

Commit message: Version enviada a JLCPCB
Parts:
- added C27: 33nF X2, Capacitor_THT:C_Rect_L11.5mm_W6.6mm_P10.00mm_MKT, F.Cu at (106.5, 93.5)
- added R29: 1M, Resistor_SMD:R_1206_3216Metric_Pad1.30x1.75mm_HandSolder, B.Cu at (122.0, 92.0)
- F1: footprint Fuse:Fuseholder_Cylinder-5x20mm_Schurter_0031_8201_Horizontal_Open -> fuente-12v:Fuseholder_BLX-A
- R1: footprint Resistor_THT:R_Axial_DIN0207_L6.3mm_D2.5mm_P10.16mm_Horizontal -> Resistor_SMD:R_1206_3216Metric_Pad1.30x1.75mm_HandSolder; moved to B.Cu
- T1: value ~ -> 750811744
- moved RV1 32.5 mm to (74.0, 85.5)
- moved FL1 24.0 mm to (89.0, 85.0)
- moved C6 19.0 mm to (79.5, 93.5), turned to 90 degrees
- moved D1 18.8 mm to (113.5, 81.0)
- moved R1 14.1 mm to (122.0, 86.0)
- moved C1 10.0 mm to (173.5, 61.8), turned to 180 degrees
- moved J2 8.50 mm to (76.0, 104.5)
- moved C5 5.56 mm to (93.0, 97.5), turned to -90 degrees
- moved J5 3.50 mm to (101.8, 124.1)
- moved F1 3.33 mm to (80.2, 75.5)
- moved C2 2.01 mm to (122.0, 81.0)
- moved C3 1.61 mm to (122.2, 68.5)
- moved C7 1.27 mm to (99.5, 107.5), turned to 90 degrees
Connections:
- C1 pad 1: P_GND -> S_GND
- C1 pad 2: SECGND -> P_GND
- C11 pad 1: SECGND -> S_GND
- C12 pad 1: SECGND -> S_GND
- C13 pad 1: SECGND -> S_GND
- C15 pad 1: SECGND -> S_GND
- C16 pad 1: SECGND -> S_GND
- C4 pad 2: SECGND -> S_GND
- C5 pad 1: Net-(C5-Pad1) -> Net-(C27-Pad2)
- C6 pad 2: Net-(C5-Pad1) -> Net-(C6-Pad2)
- C7 pad 2: /N -> Net-(C27-Pad1)
- C9 pad 2: SECGND -> S_GND
- D1 pad 2: Net-(D1-Pad2) -> Net-(C27-Pad2)
- D1 pad 3: Net-(D1-Pad3) -> Net-(C27-Pad1)
- F1 pad 2: Net-(C5-Pad1) -> Net-(C6-Pad2)
- FL1 pad 1: Net-(C5-Pad1) -> Net-(C6-Pad2)
- FL1 pad 2: Net-(D1-Pad2) -> Net-(C27-Pad2)
- FL1 pad 4: Net-(D1-Pad3) -> Net-(C27-Pad1)
- J4 pad 1: SECGND -> S_GND
- R1 pad 2: P_GND -> Net-(R1-Pad2)
- R16 pad 1: SECGND -> S_GND
- R6 pad 1: SECGND -> S_GND
- RV1 pad 1: Net-(C5-Pad1) -> Net-(C6-Pad2)
- T1 pad 12: SECGND -> S_GND
- T1 pad 13: SECGND -> S_GND
- U2 pad 4: SECGND -> S_GND
- U3 pad 3: SECGND -> S_GND
Routing:
- net SECGND: track 222.5 -> 0.00 mm
- net S_GND: track 0.00 -> 221.9 mm
- net Net-(C5-Pad1): track 84.5 -> 0.00 mm
- net Net-(C6-Pad2): track 0.00 -> 43.3 mm
- net Net-(C27-Pad2): track 0.00 -> 32.3 mm
- net /L: track 18.0 -> 42.3 mm
- net Net-(C27-Pad1): track 0.00 -> 22.2 mm
- net P_GND: track 126.1 -> 144.3 mm, vias 50 -> 48
- net /N: track 59.1 -> 41.5 mm
- net /MAINS_LINE_DC: track 43.9 -> 32.2 mm
- net Net-(D1-Pad2): track 9.39 -> 0.00 mm
- net Net-(D1-Pad3): track 9.36 -> 0.00 mm
- net +5V: track 49.8 -> 44.3 mm
- net GNDPWR: track 32.7 -> 28.4 mm
- net Net-(R1-Pad2): track 0.00 -> 2.90 mm
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Other:
- board size 150 x 85 mm -> 154 x 85 mm

Commit message: V2 routeada por bruno, necesita revision
Parts:
- removed C18, C25: 10n, Capacitor_SMD:C_0805_2012Metric_Pad1.18x1.45mm_HandSolder
- removed C26: 100nF, Capacitor_SMD:C_0805_2012Metric_Pad1.18x1.45mm_HandSolder
- removed D8, D9: 1N4148WT, Diode_SMD:D_SOD-523
- removed J3: Conn_01x03_Pin, Connector_PinHeader_2.54mm:PinHeader_1x03_P2.54mm_Vertical
- removed RV2: 1k, Potentiometer_THT:Potentiometer_Bourns_3266Y_Vertical
- removed TP3: TestPoint, Connector_PinHeader_1.00mm:PinHeader_1x01_P1.00mm_Vertical
- removed U1: NE555P, Package_DIP:DIP-8_W7.62mm
- added R30: 2M, Resistor_SMD:R_0805_2012Metric_Pad1.20x1.40mm_HandSolder, B.Cu at (161.0, 128.0)
- added R31: 2M, Resistor_SMD:R_0805_2012Metric_Pad1.20x1.40mm_HandSolder, B.Cu at (139.0, 97.0)
- added R32: 2M, Resistor_SMD:R_0805_2012Metric_Pad1.20x1.40mm_HandSolder, B.Cu at (139.0, 93.0)
- C24: value 4.7uF 50V -> 10uF 50V
- D1: footprint Diode_THT:Diode_Bridge_19.0x3.5x10.0mm_P5.0mm -> Diode_THT:Diode_Bridge_Vishay_KBL
- D5, D6: footprint Diode_SMD:D_SOD-523 -> Diode_SMD:D_SOD-323_HandSoldering
- J5: footprint Connector_PinHeader_2.54mm:PinHeader_1x02_P2.54mm_Horizontal -> Connector_PinHeader_2.54mm:PinHeader_1x02_P2.54mm_Vertical
- R27: value 220 -> 470
- R28: value 220 -> 2M
- R4: footprint Resistor_SMD:R_1206_3216Metric_Pad1.30x1.75mm_HandSolder -> Resistor_THT:R_Axial_DIN0411_L9.9mm_D3.6mm_P15.24mm_Horizontal; moved to F.Cu
- TP1, TP10, TP11, TP2, TP4, TP5, TP6, TP7, TP8, TP9: footprint Connector_PinHeader_1.00mm:PinHeader_1x01_P1.00mm_Vertical -> Connector_PinHeader_2.54mm:PinHeader_1x01_P2.54mm_Vertical
- U2: footprint Package_SO:VSSOP-8_2.3x2mm_P0.5mm -> Package_SO:Texas_S-PDSO-G8_3x3mm_P0.65mm
- moved R27 113.7 mm to (207.0, 66.0), turned to -90 degrees
- moved J5 56.7 mm to (157.5, 114.0)
- moved R28 33.5 mm to (139.0, 101.0), turned to 90 degrees
- moved R4 19.4 mm to (140.5, 69.4), turned to -90 degrees
- moved TP4 10.2 mm to (129.5, 105.0)
- moved TP10 5.59 mm to (129.5, 101.0)
- moved TP6 4.27 mm to (129.5, 109.0)
- moved H1 4.00 mm to (71.0, 130.0)
- moved H2 4.00 mm to (71.0, 55.0)
- moved D4 3.38 mm to (146.0, 77.0)
- moved C27 2.75 mm to (103.8, 93.5)
- moved C5 2.75 mm to (90.2, 97.5)
- moved C6 2.75 mm to (76.8, 93.5)
- moved C7 2.75 mm to (96.8, 107.5)
- moved D1 2.75 mm to (110.8, 81.0)
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Connections:
- J5 pad 1: P_GND -> Net-(J5-Pin_1)
- J5 pad 2: +5V -> Net-(J5-Pin_2)
- Q1 pad 1: Net-(J3-Pin_2) -> Net-(J5-Pin_1)
- R21 pad 2: Net-(J3-Pin_2) -> Net-(J5-Pin_1)
- R22 pad 1: Net-(J3-Pin_3) -> Net-(J5-Pin_2)
- R27 pad 1: +5V -> S_GND
- R27 pad 2: Net-(R27-Pad2) -> /12V
- R28 pad 1: Net-(R28-Pad1) -> Net-(U5-FLT)
- T1 pad 10: Net-(D2-A-Pad1) -> S_GND
- T1 pad 11: Net-(D2-A-Pad1) -> S_GND
- T1 pad 12: S_GND -> Net-(D2-A-Pad1)
- T1 pad 13: S_GND -> Net-(D2-A-Pad1)
- TP4 pad 1: Net-(J3-Pin_2) -> Net-(J5-Pin_1)
- U5 pad 3: unconnected-(U5-FLT-Pad3) -> Net-(U5-FLT)
Routing:
- net Net-(U5-FLT): track 0.00 -> 68.1 mm, vias 0 -> 2
- net /AUX_DRV: track 64.4 -> 0.00 mm
- net +5V: track 44.3 -> 0.00 mm
- net Net-(J5-Pin_1): track 0.00 -> 37.1 mm, vias 0 -> 1
- net /TRIG: track 35.3 -> 0.00 mm
- net Net-(J3-Pin_2): track 26.3 -> 0.00 mm
- net /VOUT: track 14.6 -> 5.02 mm
- net /DIS: track 9.08 -> 0.00 mm
- net Net-(D6-K): track 59.5 -> 65.3 mm
- net Net-(U1-CV): track 4.95 -> 0.00 mm
- net Net-(D2-A-Pad1): track 59.2 -> 63.9 mm
- net S_GND: track 221.9 -> 217.9 mm
- net Net-(C14-Pad2): track 6.09 -> 9.91 mm
- net Net-(R27-Pad2): track 3.70 -> 0.00 mm
- net Net-(Q1-S): track 24.3 -> 27.7 mm
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- added copper zone on B.Cu, net /LINE_DC
- added copper zone on B.Cu, net /VOUT
- added copper zone on B.Cu, net Net-(D2-A-Pad1)
- added copper zone on B.Cu, net Net-(D4-A)
- added copper zone on B.Cu, net S_GND
Other:
- board text added: "Fuente Flyback 12V 2.5A V2 Proyecto Electrónica de Potencia 2025"
- board text removed: "Fuente Flyback 12V 2.5A Proyecto Electrónica de Potenica 2025"
- board text removed: "VOUT"

Commit message: Cambios v2
Parts:
- R4: value 80k -> 27k
- R5, R8: value 0.018 -> 0.047
- moved R5 0.11 mm to (210.1, 73.0)
Connections:
- C13 pad 2: /12V -> /12V_FILT
- C15 pad 2: Net-(D2-K) -> /12V
- C16 pad 2: Net-(D2-K) -> /12V
- C17 pad 2: Net-(D2-K) -> /12V
- C4 pad 1: /12V -> /12V_FILT
- C9 pad 1: Net-(D2-K) -> /12V
- D2 pad 2: Net-(D2-K) -> /12V
- L1 pad 1: Net-(D2-K) -> /12V
- L1 pad 2: /12V -> /12V_FILT
- R2 pad 1: /12V -> /12V_FILT
- R27 pad 2: /12V -> /12V_FILT
- R5 pad 2: /12V -> /12V_FILT
- R7 pad 2: /12V -> /12V_FILT
- R8 pad 2: /12V -> /12V_FILT
- TP2 pad 1: /12V -> /12V_FILT
- U2 pad 8: /12V -> /12V_FILT
Routing:
- net /12V_FILT: track 0.00 -> 80.5 mm
- net /12V: track 144.7 -> 74.8 mm
- net Net-(D2-K): track 51.2 -> 0.00 mm
- net S_GND: track 217.9 -> 197.1 mm, vias 0 -> 1
- net P_GND: track 145.8 -> 145.1 mm
Other:
- board text added: "Fuente Flyback 12V 2A V2 Proyecto Electrónica de Potencia 2025"
- board text removed: "Fuente Flyback 12V 2.5A V2 Proyecto Electrónica de Potencia 2025"

Commit message: V2 fabricada
Parts:
- added TP12: TestPoint, Connector_PinHeader_2.54mm:PinHeader_1x01_P2.54mm_Vertical, F.Cu at (161.5, 117.7)
- added TP13: TestPoint, Connector_PinHeader_2.54mm:PinHeader_1x01_P2.54mm_Vertical, F.Cu at (209.8, 105.3)
- added TP14: TestPoint, Connector_PinHeader_2.54mm:PinHeader_1x01_P2.54mm_Vertical, F.Cu at (156.5, 127.8)
- added TP3: TestPoint, Connector_PinHeader_2.54mm:PinHeader_1x01_P2.54mm_Vertical, F.Cu at (129.5, 112.7)
- R25: value 0.47 -> DNP
- R26: value 10k -> 1k
- R5: value 0.047 -> DNP
- moved TP11 7.29 mm to (161.5, 113.7), turned to 0 degrees
- moved C8 5.35 mm to (135.0, 93.7)
- moved TP10 5.20 mm to (129.4, 95.8), turned to 0 degrees
- moved TP4 3.70 mm to (129.4, 101.3)
- moved TP6 1.90 mm to (129.5, 107.1)
- moved TP7 0.15 mm to (209.9, 114.0), turned to 0 degrees
Routing:
- net S_GND: track 197.1 -> 206.3 mm
- net /VAUX: track 25.3 -> 34.3 mm
- net P_GND: track 145.1 -> 152.7 mm, vias 35 -> 34
- net Net-(D6-A): track 33.2 -> 38.5 mm
- net Net-(D6-K): track 65.3 -> 69.1 mm
- net Net-(U5-CS): track 26.9 -> 28.9 mm
- net Net-(J5-Pin_1): track 37.1 -> 38.7 mm
- net Net-(U5-FLT): track 68.1 -> 68.9 mm
- net Net-(Q1-S): track 27.7 -> 28.3 mm
Other:
- outline, holes or cut-outs redrawn
- board text added: "CS_UCC"
- board text added: "P_GND"
- board text added: "S_GND"
